Commit message: added g1 to scene

File: dexmachina/assets/xhand/xhand_left_6dof.urdf (robot description, URDF)
Before this commit: robot xhand_left, 25 links, 24 joints
Joints:
- joint L_forearm_tx_link_joint: limit lower=-5.0 upper=5.0 effort=100 velocity=5 -> lower=-2.0 upper=2.0 effort=100 velocity=5
- joint L_forearm_ty_link_joint: limit lower=-5.0 upper=5.0 effort=100 velocity=5 -> lower=-2.0 upper=2.0 effort=100 velocity=5
- joint L_forearm_tz_link_joint: limit lower=-5.0 upper=5.0 effort=100 velocity=5 -> lower=-2.0 upper=2.0 effort=100 velocity=5
